File: solenoid.kicad_sch (KiCad schematic)
At the start: 5 parts, among them J3 B2B-PH-K-S(LF)(SN), Q3 BSS138

Commit message: a
Parts:
- removed J3: B2B-PH-K-S(LF)(SN), Connector_JST:JST_PH_B2B-PH-K_1x02_P2.00mm_Vertical, symbol Connector:Conn_01x02_Pin
- removed R3: 1k, Resistor_SMD:R_0603_1608Metric, symbol Device:R
- added C2: 1000u, Capacitor_THT:CP_Radial_D10.0mm_P5.00mm, symbol Device:C_Polarized
- renumbered D3 to D1, Q3 to Q1, S3 to S1
Connections:
- net +24V: now also C2.1
- net GND: now also C2.2
