File: solenoid_board.kicad_pcb (KiCad board)
At the start: 2 copper layers, 30 x 70 mm, 45 parts, among them J1 B2B-PH-K-S(LF)(SN), J10 Conn_01x02_Pin, J2 B2B-PH-K-S(LF)(SN), J3 B2B-PH-K-S(LF)(SN), J4 B2B-PH-K-S(LF)(SN), J5 B2B-PH-K-S(LF)(SN), J6 B2B-PH-K-S(LF)(SN), J7 B2B-PH-K-S(LF)(SN), J8 B2B-PH-K-S(LF)(SN), J9 C5665, Q1 BSS138, Q2 BSS138, Q3 BSS138, Q4 BSS138, Q5 BSS138, Q6 BSS138, Q7 BSS138, Q8 BSS138

Commit message: a
Parts:
- removed J3, J4, J5, J6, J7, J8: B2B-PH-K-S(LF)(SN), Connector_JST:JST_PH_B2B-PH-K_1x02_P2.00mm_Vertical
- removed R8: 1k, Resistor_SMD:R_0603_1608Metric
- added C2: 1000u, Capacitor_THT:CP_Radial_D10.0mm_P5.00mm, F.Cu at (180.8, 25.4)
- added C3: 1000u, Capacitor_THT:CP_Radial_D10.0mm_P5.00mm, F.Cu at (172.4, 32.0)
- added C4: 1000u, Capacitor_THT:CP_Radial_D10.0mm_P5.00mm, F.Cu at (180.8, 39.2)
- added C5: 1000u, Capacitor_THT:CP_Radial_D10.0mm_P5.00mm, F.Cu at (172.4, 46.4)
- added C6: 1000u, Capacitor_THT:CP_Radial_D10.0mm_P5.00mm, F.Cu at (180.8, 53.6)
- added C7: 1000u, Capacitor_THT:CP_Radial_D10.0mm_P5.00mm, F.Cu at (172.4, 60.8)
- added C8: 1000u, Capacitor_THT:CP_Radial_D10.0mm_P5.00mm, F.Cu at (180.8, 68.2)
- added C9: 1000u, Capacitor_THT:CP_Radial_D10.0mm_P5.00mm, F.Cu at (172.4, 75.4)
- added D10: LED, LED_SMD:LED_0603_1608Metric, F.Cu at (107.2, 30.0)
- added D11: LED, LED_SMD:LED_0603_1608Metric, F.Cu at (107.2, 40.0)
- added D12: LED, LED_SMD:LED_0603_1608Metric, F.Cu at (107.2, 50.0)
- added D13: LED, LED_SMD:LED_0603_1608Metric, F.Cu at (107.2, 60.0)
- added D14: LED, LED_SMD:LED_0603_1608Metric, F.Cu at (107.2, 70.0)
- added D15: LED, LED_SMD:LED_0603_1608Metric, F.Cu at (107.2, 80.0)
- added D16: LED, LED_SMD:LED_0603_1608Metric, F.Cu at (107.2, 90.0)
- J1: value B2B-PH-K-S(LF)(SN) -> Conn_01x10_Pin; footprint Connector_JST:JST_PH_B2B-PH-K_1x02_P2.00mm_Vertical -> Connector_PinSocket_2.54mm:PinSocket_1x10_P2.54mm_Vertical
- J2: value B2B-PH-K-S(LF)(SN) -> Conn_01x10_Socket; footprint Connector_JST:JST_PH_B2B-PH-K_1x02_P2.00mm_Vertical -> Connector_PinHeader_2.54mm:PinHeader_1x10_P2.54mm_Horizontal
- R1, R2, R3, R4, R5, R6, R7: value 1k -> R
- moved D9 70.9 mm to (177.9, 98.7)
- moved R9 70.9 mm to (181.4, 98.7)
- moved C1 44.5 mm to (165.4, 82.8), turned to 180 degrees
- moved J10 42.2 mm to (175.7, 86.2), turned to 90 degrees
- moved J9 38.3 mm to (159.9, 95.8), turned to 90 degrees
- moved R7 34.7 mm to (131.2, 63.8), turned to 180 degrees
- moved R6 32.4 mm to (131.2, 61.2), turned to 180 degrees
- moved R1 31.6 mm to (131.2, 48.6), turned to 180 degrees
- moved R5 30.8 mm to (131.2, 58.6), turned to 180 degrees
- moved R2 30.5 mm to (131.2, 51.2), turned to 180 degrees
- moved R4 30.0 mm to (131.2, 56.0), turned to 180 degrees
- moved R3 29.8 mm to (131.2, 53.6), turned to 180 degrees
- moved J2 29.0 mm to (135.0, 48.6), turned to 0 degrees
- moved D8 19.5 mm to (160.1, 76.5)
- moved D7 19.3 mm to (160.1, 69.2)
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Connections:
- J1 pad 1: GND -> /S1
- J1 pad 2: Net-(J1-Pin_2) -> /S2
- J2 pad 1: GND -> Net-(J2-Pin_1)
- J9 pad 1: +24V -> unconnected-(J9-Pin_1-Pad1)
- R1 pad 1: /S1 -> Net-(J2-Pin_1)
- R1 pad 2: Net-(J1-Pin_2) -> Net-(D10-A)
- R2 pad 1: /S2 -> Net-(J2-Pin_2)
- R2 pad 2: Net-(J2-Pin_2) -> Net-(D11-A)
- R3 pad 1: /S3 -> Net-(J2-Pin_3)
- R4 pad 1: /S4 -> Net-(J2-Pin_4)
- R5 pad 1: /S5 -> Net-(J2-Pin_5)
- R6 pad 1: /S6 -> Net-(J2-Pin_6)
- R7 pad 1: /S7 -> Net-(J2-Pin_7)
Routing:
- net Net-(D10-K): track 0.00 -> 101.5 mm, vias 0 -> 7
- net /S2: track 26.0 -> 85.8 mm, vias 0 -> 1
- net /S3: track 23.3 -> 79.6 mm, vias 0 -> 1
- net /S4: track 14.7 -> 63.9 mm, vias 0 -> 1
- net /S1: track 35.4 -> 82.1 mm
- net /S5: track 15.7 -> 57.5 mm, vias 0 -> 1
- net Net-(D16-A): track 3.02 -> 35.5 mm
- net Net-(D10-A): track 0.00 -> 31.2 mm
- net /S6: track 18.1 -> 47.0 mm, vias 0 -> 1
- net Net-(D11-A): track 0.00 -> 28.1 mm
- net Net-(D15-A): track 3.02 -> 30.6 mm
- net Net-(D14-A): track 3.07 -> 27.6 mm
- net Net-(D12-A): track 3.48 -> 25.0 mm
- net Net-(D13-A): track 3.16 -> 24.5 mm
- net /S7: track 26.8 -> 45.6 mm, vias 0 -> 1
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- added copper zone on F.Cu, net GND
Other:
- board size 30 x 70 mm -> 86 x 80 mm
- board text added: "Solenoid driver board v0.2.0 designed by mmaakkyyii"
- board text removed: "Solenoid driver board v0.1.0 designed by mmaakkyyii"
