File: solenoid_board.kicad_sch (KiCad schematic)
At the start: 5 parts, among them J10 Conn_01x02_Pin, J9 C5665

Commit message: a
Parts:
- added D10, D11, D12, D13, D14, D15, D16: LED, LED_SMD:LED_0603_1608Metric, symbol Device:LED
- added J1: Conn_01x10_Pin, Connector_PinSocket_2.54mm:PinSocket_1x10_P2.54mm_Vertical, symbol Connector:Conn_01x10_Pin
- added J2: Conn_01x10_Socket, Connector_PinHeader_2.54mm:PinHeader_1x10_P2.54mm_Horizontal, symbol Connector:Conn_01x10_Socket
- added R1, R2, R3, R4, R5, R6, R7: R, Resistor_SMD:R_0603_1608Metric, symbol Device:R
- D9: JLCPCB Parts# (none) -> C273617
Connections:
- net +24V: no longer J9.1 (Pin_1)
- net GND: now also J1.9 (Pin_9)
- net S1: now also J1.1 (Pin_1)
- net S2: now also J1.2 (Pin_2)
- net S3: now also J1.3 (Pin_3)
- net S4: now also J1.4 (Pin_4)
- net S5: now also J1.5 (Pin_5)
- net S6: now also J1.6 (Pin_6)
- net S7: now also J1.7 (Pin_7)
- net S8: now also J1.8 (Pin_8)
- new net: J2.5 (Pin_5), R5.1
- new net: D14.2 (A), R5.2
- new net: D10.1 (K), D11.1 (K), D12.1 (K), D13.1 (K), D14.1 (K), D15.1 (K), D16.1 (K), J2.9 (Pin_9)
- new net: D10.2 (A), R1.2
- new net: D13.2 (A), R4.2
- new net: J2.1 (Pin_1), R1.1
- new net: D11.2 (A), R2.2
- new net: D12.2 (A), R3.2
- new net: J2.2 (Pin_2), R2.1
- new net: D15.2 (A), R6.2
- new net: J2.6 (Pin_6), R6.1
- new net: J2.3 (Pin_3), R3.1
- new net: J2.7 (Pin_7), R7.1
- new net: D16.2 (A), R7.2
- new net: J2.4 (Pin_4), R4.1
- no-connect marks 0 -> 1
